File: hardware/soilboard/soilboard.kicad_sch (KiCad schematic)
At the start: 73 parts, among them IC1 TP4056, J1 USB_C_Receptacle_USB2.0, J10 Conn_01x03, J11 Conn_01x02_Female, J12 Conn_01x06, J13 Conn_01x06, J14 Conn_01x02, J15 Conn_01x06, J16 Conn_01x06, J2 Conn_01x04, J3 Conn_01x04, J4 Conn_01x04, J5 Conn_01x03, J6 Conn_01x03, J7 Conn_01x02_Female, J8 Conn_01x03, J9 JST XH 2P 2.50mm SMD Hoz, SW1 Tactile Switch 3x4x2, SW2 Tactile Switch 3x4x2, SW3 MST22D18G2_125, T1 IRLML6344TRPBF, T2 IRLML6344TRPBF, U1 CH340K, U2 AO3401A, U3 SPX3819M5-L-3-3/TR, U4 2N27002DW, U5 ESP32-S3-WROOM-1

Commit message: Delete USB-UART interface which is no longer needed with ESP32-s3. Add eletrostatic discharge protection.
Parts:
- removed C3: 100nF, Capacitor_SMD:C_0603_1608Metric, symbol Device:C
- removed J12: Conn_01x06, Connector_PinHeader_2.54mm:PinHeader_1x06_P2.54mm_Vertical, symbol Connector_Generic:Conn_01x06
- removed R7, R8: 1K, Resistor_SMD:R_0603_1608Metric, symbol Device:R
- removed U1: CH340K, DroneV2:ESSOP-10_3.9x4.9mm_P1.00mm, symbol downloader-rescue:ch340k-my
- removed U4: 2N27002DW, Package_TO_SOT_SMD:SOT-363_SC-70-6, symbol downloader-rescue:DDC114TU-7-F-my
- added J12: Conn_01x04, Connector_PinHeader_2.54mm:PinHeader_1x04_P2.54mm_Vertical, symbol Connector_Generic:Conn_01x04
- added R24, R25: 10k, Resistor_SMD:R_0603_1608Metric, symbol Device:R
- added U3: USBLC6-2SC6, Package_TO_SOT_SMD:SOT-23-6, symbol Power_Protection:USBLC6-2SC6
- C1: value 100nF -> 1 uF; JLCA Type Basic -> (none); LCSC Link https://www.lcsc.com/product-detail/Multilayer-Ceramic-Capa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 -> (none); LCSC Part # C14663 -> (none); MFR.Part # CC0603KRX7R9BB104 -> (none); Manufacturer YAGEO -> (none); Package C0603 -> (none)
- renumbered C11 to C10, C12 to C11, C4 to C3, C5 to C4, C6 to C5, C7 to C6, C8 to C7, C9 to C8, C10 to C9, R3 to R1, R12 to R10, R13 to R11, R14 to R12, R15 to R13, R16 to R14, R17 to R15, R18 to R16, R19 to R17, R20 to R18, R21 to R19, R4 to R2, R22 to R20, R23 to R21, R24 to R22, R25 to R23, R5 to R3, R1 to R4, R2 to R5, R9 to R7, R10 to R8, R11 to R9, U2 to U1, U3 to U2, U5 to U4
Connections:
- net D+: now also U3.1 (I/O1)
- net D-: now also U3.3 (I/O2)
- net GND: now also C1.2, R24.1, R25.1, U3.2 (GND); no longer C1.1
- net IO17: now also J12.1 (Pin_1)
- net IO18: now also J12.2 (Pin_2)
- net IO21: now also J12.3 (Pin_3)
- net IO47: now also J12.4 (Pin_4)
- net RX: now also R24.2
- net TX: now also R25.2
- net VBUS: now also C1.1, U3.5 (VBUS)
- net IO19 renamed D_PROC-
- net D_PROC-: now also U3.4 (I/O2)
- net IO20 renamed D_PROC+
- net D_PROC+: now also U3.6 (I/O1)
- no-connect marks 5 -> 4
Other:
- note added: "ESD Protection"
- note removed: "Auto Reset Circuit"
- note removed: "USB - UART / Programming Circuit"
- moved on the sheet: LED1, LED2, LED3, R1, R2, R3

Commit message: SOILBoard v0.3 send off for manufacturing.
Parts:
- removed J11, J7: Conn_01x02_Female, DroneV2:JST_PH_B2B-PH-K_1x02_P2.00mm_Vertical, symbol Connector:Conn_01x02_Female
- removed J12: Conn_01x04, Connector_PinHeader_2.54mm:PinHeader_1x04_P2.54mm_Vertical, symbol Connector_Generic:Conn_01x04
- removed J13, J15, J16: Conn_01x06, Connector_PinHeader_2.54mm:PinHeader_1x06_P2.54mm_Vertical, symbol Connector_Generic:Conn_01x06
- removed J14: Conn_01x02, DroneV2:CONN-TH_1.25T-2A_1.25T-2A, symbol Connector_Generic:Conn_01x02
- removed R15, R16, R24, R25: 10k, Resistor_SMD:R_0603_1608Metric, symbol Device:R
- added J11, J7: Conn_01x02_Socket, TerminalBlock:TerminalBlock_bornier-2_P5.08mm, symbol Connector:Conn_01x02_Socket
- added J12: Conn_01x09_Socket, Connector_PinSocket_2.54mm:PinSocket_1x09_P2.54mm_Vertical, symbol Connector:Conn_01x09_Socket
- added J13: Extra_01x04_Socket, Connector_PinHeader_2.54mm:PinHeader_1x05_P2.54mm_Vertical, symbol Connector:Conn_01x05_Socket
- J2: value Conn_01x04 -> Temp_01x04
- J3: value Conn_01x04 -> Ping_01x04
- J4: value Conn_01x04 -> Stemma_01x04
- renumbered R17 to R15, R18 to R16, R19 to R17, R20 to R18, R21 to R19, R22 to R20, R23 to R21
Connections:
- net CLK is gone; now on net SOIL2: U4.29 (IO36)
- net IO1 is gone; now on net SCL1: U4.39 (IO1)
- net IO21 is gone; now on net SERVO2: U4.23 (IO21)
- net IO47 is gone; now on net LED_GREEN: U4.24 (IO47)
- net IO48 is gone; now on net LED_RED: U4.25 (IO48)
- net +3V3: now also J12.9 (Pin_9)
- net +BATT: now also J11.1 (Pin_1), J7.1 (Pin_1)
- net ADC_BAT: now also U4.30 (IO37); no longer U4.38 (IO2)
- net CS: now also U4.15 (IO3), J12.7 (Pin_7); no longer U4.35 (IO42)
- net ECHO: now also U4.4 (IO4); no longer U4.22 (IO14)
- net GND: now also R12.2, J12.8 (Pin_8); no longer R12.1
- net IO17: now also J13.3 (Pin_3)
- net IO18: now also J13.4 (Pin_4)
- net LED_BLUE: now also U4.26 (IO45); no longer U4.7 (IO7)
- net LED_GREEN: no longer U4.17 (IO9)
- net LED_RED: no longer U4.12 (IO8)
- net MISO: now also U4.22 (IO14), J12.1 (Pin_1); no longer U4.30 (IO37)
- net MOSI: now also U4.18 (IO10), J12.4 (Pin_4); no longer U4.28 (IO35)
- net SCL1: no longer U4.34 (IO41)
- net SCL2: now also R15.1, U4.35 (IO42); no longer U4.9 (IO16)
- net SDA1: now also U4.38 (IO2); no longer U4.33 (IO40)
- net SDA2: now also R16.1, U4.34 (IO41); no longer U4.8 (IO15)
- net SERVO1: now also U4.21 (IO13); no longer U4.15 (IO3)
- net SERVO2: no longer U4.4 (IO4)
- net SOIL1: now also U4.6 (IO6); no longer U4.26 (IO45)
- net SOIL2: no longer U4.16 (IO46)
- net TRIG: now also U4.5 (IO5); no longer U4.21 (IO13)
- net at C6.2, D2.2 (A), T1.3 (D): now also J7.2 (Pin_2)
- net at C8.2, D3.2 (A), T2.3 (D): now also J11.2 (Pin_2)
- net BUZ1: no longer names the net of U4.31 (IO38)
- net BUZ2: no longer names the net of U4.32 (IO39)
- net IO12 renamed LED_TFT
- net LED_TFT: now also J12.2 (Pin_2)
- net MOT_1 renamed MOT1
- net MOT1: now also U4.7 (IO7); no longer U4.5 (IO5)
- removed net MOT_2: R12.2, T2.1 (G), U4.6 (IO6)
- net RX: no longer names the net of U4.36 (RXD0)
- removed net SCL: R16.1, U4.18 (IO10)
- net SDA renamed SCK
- net SCK: now also J12.3 (Pin_3); no longer R15.1
- net TX: no longer names the net of U4.37 (TXD0)
- new net DC: J12.5 (Pin_5), U4.17 (IO9)
- new net IO15: J13.1 (Pin_1), U4.8 (IO15)
- new net IO16: J13.2 (Pin_2), U4.9 (IO16)
- new net IO8: J13.5 (Pin_5), U4.12 (IO8)
- new net MOT2: R12.1, T2.1 (G), U4.28 (IO35)
- new net RESET: J12.6 (Pin_6), U4.16 (IO46)
- no-connect marks 4 -> 9
Other:
- note added: "(Optional) ILI9341 TFT display"
- note added: "Extra Expansion"
- note removed: "Debugger"
- note removed: "Leftover Pins"
- note removed: "SPI Expansion"
- note removed: "UART/I2C Expansion"
- moved on the sheet: C3, R12, R20, R21
